Commit message: made  change

File: description/robot_core.xacro (robot description, xacro)
@@ -22,7 +22,7 @@
     <link name="chasis">
         <visual>
-            <origin xyz="0.15 0 0.075"/>
+            <origin xyz="0.3 0 0.075"/>
             <geometry>
-                <box_size="0.6 0.6 0.15"/>
+                <box size="0.6 0.6 0.15"/>
             </geometry>
             <material name="white"/>

Commit message: change

File: description/robot_core.xacro (robot description, xacro)
@@ -24,5 +24,4 @@
             <origin xyz="0.3 0 0.075"/>
             <geometry>
-                <box size="0.6 0.6 0.15"/>
             </geometry>
             <material name="white"/>

Commit message: change

File: description/robot_core.xacro (robot description, xacro)
@@ -24,4 +24,5 @@
             <origin xyz="0.3 0 0.075"/>
             <geometry>
+                <box size ="0.6 0.6 0.15"/>
             </geometry>
             <material name="white"/>

Commit message: change

File: description/robot_core.xacro (robot description, xacro)
@@ -1,4 +1,4 @@
 <?xml version="1.0"?>
-<robot xmlns:xacro="http://www.ros.org/wiki/xacro">
+<robot xmlns:xacro="http://www.ros.org/wiki/xacro" >
     <material name="white">
         <color rgba="1 1 1 1"/>
@@ -13,5 +13,5 @@
         <color rgba="0 0 0 1"/>
     </material>
-    <link_name="base_link">
+    <link name="base_link">
     </link>
     <joint name="chassis_joint" type="fixed">

Commit message: change

File: description/robot_core.xacro (robot description, xacro)
@@ -20,5 +20,5 @@
         <orgin xyz="-0.1 0 0"/>
     </joint>
-    <link name="chasis">
+    <link name="chassis">
         <visual>
             <origin xyz="0.3 0 0.075"/>

Commit message: change

File: description/robot_core.xacro (robot description, xacro)
@@ -18,5 +18,5 @@
         <parent link="base_link"/>
         <child link="chassis"/>
-        <orgin xyz="-0.1 0 0"/>
+        <origin xyz="-0.1 0 0"/>
     </joint>
     <link name="chassis">

Commit message: change

File: description/robot_core.xacro (robot description, xacro)
@@ -1,15 +1,6 @@
 <?xml version="1.0"?>
-<robot xmlns:xacro="http://www.ros.org/wiki/xacro" >
+<robot xmlns:xacro="http://www.ros.org/wiki/xacro">
     <material name="white">
         <color rgba="1 1 1 1"/>
-    </material>
-    <material name="orange">
-        <color rgba="1 0.3 0.1 1"/>
-    </material>
-    <material name="blue">
-        <color rgba="0.2 0.2 1 1"/>
-    </material>
-    <material name="black">
-        <color rgba="0 0 0 1"/>
     </material>
     <link name="base_link">
@@ -24,8 +15,19 @@
             <origin xyz="0.3 0 0.075"/>
             <geometry>
-                <box size ="0.6 0.6 0.15"/>
+                <box size="0.6 0.6 0.15"/>
             </geometry>
             <material name="white"/>
         </visual>
+        <collision>
+            <origin xyz="0.3 0 0.075"/>
+            <geometry>
+                <box size="0.6 0.6 0.15"/>
+            </geometry>
+        </collision>
+        <inertial>
+            <mass value="1.0"/>
+            <origin xyz="0 0 0"/>
+            <inertia ixx="0.1" ixy="0" ixz="0" iyy="0.1" iyz="0" izz="0.1"/>
+        </inertial>
     </link>
 </robot>

Commit message: change

File: description/robot_core.xacro (robot description, xacro)
@@ -1,6 +1,15 @@
 <?xml version="1.0"?>
-<robot xmlns:xacro="http://www.ros.org/wiki/xacro">
+<robot xmlns:xacro="http://www.ros.org/wiki/xacro" >
     <material name="white">
         <color rgba="1 1 1 1"/>
+    </material>
+    <material name="orange">
+        <color rgba="1 0.3 0.1 1"/>
+    </material>
+    <material name="blue">
+        <color rgba="0.2 0.2 1 1"/>
+    </material>
+    <material name="black">
+        <color rgba="0 0 0 1"/>
     </material>
     <link name="base_link">
@@ -15,19 +24,8 @@
             <origin xyz="0.3 0 0.075"/>
             <geometry>
-                <box size="0.6 0.6 0.15"/>
+                <box size ="0.6 0.6 0.15"/>
             </geometry>
             <material name="white"/>
         </visual>
-        <collision>
-            <origin xyz="0.3 0 0.075"/>
-            <geometry>
-                <box size="0.6 0.6 0.15"/>
-            </geometry>
-        </collision>
-        <inertial>
-            <mass value="1.0"/>
-            <origin xyz="0 0 0"/>
-            <inertia ixx="0.1" ixy="0" ixz="0" iyy="0.1" iyz="0" izz="0.1"/>
-        </inertial>
     </link>
 </robot>

Commit message: change

File: description/robot_core.xacro (robot description, xacro)
@@ -22,7 +22,7 @@
     <link name="chassis">
         <visual>
-            <origin xyz="0.3 0 0.075"/>
+            <origin xyz="0.15 0 0.075"/>
             <geometry>
-                <box size ="0.6 0.6 0.15"/>
+                <box size ="0.3 0.3 0.15"/>
             </geometry>
             <material name="white"/>

Commit message: change

File: description/robot_core.xacro (robot description, xacro)
@@ -29,3 +29,16 @@
         </visual>
     </link>
+    <joint name="left_wheel_joint" type="continous">
+        <parent link="base_link"/>
+        <child link="chassis"/>
+        <orgin xyz="0 0.175 0" rpy="-${pi/2} 0 0"/>
+    </joint>
+    <link name="left_wheel">
+        <visual>
+            <geometry>
+                <cylinder radius ="0.05" length-"0.04"/>
+            </geometry>
+            <material name="blue"/>
+        </visual>
+    </link>
 </robot>

Commit message: change

File: description/robot_core.xacro (robot description, xacro)
@@ -1,4 +1,5 @@
 <?xml version="1.0"?>
 <robot xmlns:xacro="http://www.ros.org/wiki/xacro" >
+    <xacro:include filename="intertial_macros.xacro"/>
     <material name="white">
         <color rgba="1 1 1 1"/>
@@ -29,16 +30,50 @@
         </visual>
     </link>
+        <collision>
+            <origin xyz="0.15 0 0.075"/>
+            <geometry>
+                <box size ="0.3 0.3 0.15"/>
+            </geometry>
+        </collision>
+        <xacro:inertial_box mass="0.5" x="0.3" y="0.3" z="0.15">
+            <orgin xyz="0.15 0 0.075" rpy="0 0 0"/>
+    </link>
     <joint name="left_wheel_joint" type="continous">
         <parent link="base_link"/>
-        <child link="chassis"/>
+        <child link="left_wheel"/>
         <orgin xyz="0 0.175 0" rpy="-${pi/2} 0 0"/>
+        <axis xyz="0 0 1"/>
     </joint>
     <link name="left_wheel">
         <visual>
             <geometry>
-                <cylinder radius ="0.05" length-"0.04"/>
+                <cylinder radius ="0.05" length="0.04"/>
             </geometry>
             <material name="blue"/>
         </visual>
+        <collission>
+            <geometry>
+                <cylinder radius ="0.05" length="0.04"/>
+            </geometry>
+        </collision>
+    </link>
+    <joint name="right_wheel_joint" type="continous">
+        <parent link="base_link"/>
+        <child link="right_wheel"/>
+        <orgin xyz="0 -0.175 0" rpy="${pi/2} 0 0"/>
+        <axis xyz="0 0 -1"/>
+    </joint>
+    <link name="right_wheel">
+        <visual>
+            <geometry>
+                <cylinder radius ="0.05" length="0.04"/>
+            </geometry>
+            <material name="blue"/>
+        </visual>
+        <collision>
+            <geometry>
+                <cylinder radius ="0.05" length="0.04"/>
+            </geometry>
+        </collision>
     </link>
 </robot>

Commit message: change

File: description/robot_core.xacro (robot description, xacro)
@@ -29,5 +29,4 @@
             <material name="white"/>
         </visual>
-    </link>
         <collision>
             <origin xyz="0.15 0 0.075"/>
@@ -37,34 +36,14 @@
         </collision>
         <xacro:inertial_box mass="0.5" x="0.3" y="0.3" z="0.15">
-            <orgin xyz="0.15 0 0.075" rpy="0 0 0"/>
+            <origin xyz="0.15 0 0.075" rpy="0 0 0"/>
     </link>
-    <joint name="left_wheel_joint" type="continous">
+    <!-- LEFT WHEEL LINK -->
+    <joint name="left_wheel_joint" type="continuous">
         <parent link="base_link"/>
         <child link="left_wheel"/>
-        <orgin xyz="0 0.175 0" rpy="-${pi/2} 0 0"/>
+        <origin xyz="0 0.175 0" rpy="-${pi/2} 0 0"/>
         <axis xyz="0 0 1"/>
     </joint>
     <link name="left_wheel">
-        <visual>
-            <geometry>
-                <cylinder radius ="0.05" length="0.04"/>
-            </geometry>
-            <material name="blue"/>
-        </visual>
-        <collission>
-            <geometry>
-                <cylinder radius ="0.05" length="0.04"/>
-            </geometry>
-        </collision>
-        <xacro:inertial_cylinder mass="0.1" length="0.04" radius="0.02">
-            <orgin xyz="0"
-    </link>
-    <joint name="right_wheel_joint" type="continous">
-        <parent link="base_link"/>
-        <child link="right_wheel"/>
-        <orgin xyz="0 -0.175 0" rpy="${pi/2} 0 0"/>
-        <axis xyz="0 0 -1"/>
-    </joint>
-    <link name="right_wheel">
         <visual>
             <geometry>
@@ -78,4 +57,20 @@
             </geometry>
         </collision>
+        <xacro:inertial_cylinder mass="0.1" length="0.04" radius="0.02">
+            <orgin xyz="0"
+    </link>
+    <joint name="right_wheel_joint" type="continuous">
+        <parent link="base_link"/>
+        <child link="right_wheel"/>
+        <origin xyz="0 -0.175 0" rpy="${pi/2} 0 0"/>
+        <axis xyz="0 0 -1"/>
+    </joint>
+    <link name="right_wheel">
+        <visual>
+            <geometry>
+                <cylinder radius ="0.05" length="0.04"/>
+            </geometry>
+            <material name="blue"/>
+        </visual>
     </link>
 </robot>

Commit message: change

File: description/robot_core.xacro (robot description, xacro)
@@ -35,6 +35,4 @@
             </geometry>
         </collision>
-        <xacro:inertial_box mass="0.5" x="0.3" y="0.3" z="0.15">
-            <origin xyz="0.15 0 0.075" rpy="0 0 0"/>
     </link>
     <!-- LEFT WHEEL LINK -->
@@ -57,6 +55,4 @@
             </geometry>
         </collision>
-        <xacro:inertial_cylinder mass="0.1" length="0.04" radius="0.02">
-            <orgin xyz="0"
     </link>
     <joint name="right_wheel_joint" type="continuous">
@@ -73,4 +69,9 @@
             <material name="blue"/>
         </visual>
+        <collision>
+            <geometry>
+                <cylinder radius ="0.05" length="0.04"/>
+            </geometry>
+        </collision>
     </link>
 </robot>

Commit message: change

File: description/robot_core.xacro (robot description, xacro)
@@ -1,4 +1,5 @@
 <?xml version="1.0"?>
 <robot xmlns:xacro="http://www.ros.org/wiki/xacro" >
+    <xacro:include filename="inertial_macros.xacro"/>
     <material name="white">
         <color rgba="1 1 1 1"/>
@@ -37,4 +38,6 @@
             </geometry>
         </collision>
+        <xacro:inertial_box mass="0.5" x="0.3" y="0.3" z="0.15">
+            <origin xyz="-0.1 0 0" rpy="0 0 0"/>
     </link>
     <!-- LEFT WHEEL LINK -->
@@ -57,4 +60,7 @@
             </geometry>
         </collision>
+        <xacro:inertial_cylinder mass="0.1" length="0.04" radius="0.05">
+            <origin xyz="0 0 0" rpy="0 0 0"/>
+        </xacro:inertial_cylinder>
     </link>
     <joint name="right_wheel_joint" type="continuous">
@@ -76,4 +82,7 @@
             </geometry>
         </collision>
+        <xacro:inertial_cylinder mass="0.1" length="0.04" radius="0.05">
+            <origin xyz="0 0 0" rpy="0 0 0"/>
+        </xacro:inertial_cylinder>
     </link>
 </robot>

Commit message: change

File: description/robot_core.xacro (robot description, xacro)
@@ -39,5 +39,6 @@
         </collision>
         <xacro:inertial_box mass="0.5" x="0.3" y="0.3" z="0.15">
-            <origin xyz="-0.1 0 0" rpy="0 0 0"/>
+            <origin xyz="-0.15 0 0.075" rpy="0 0 0"/>
+        </xacro:inertial_box>
     </link>
     <!-- LEFT WHEEL LINK -->

Commit message: change

File: description/robot_core.xacro (robot description, xacro)
@@ -33,18 +33,18 @@
     <link name="chassis">
         <visual>
-            <origin xyz="0.15 0 0.075"/>
+            <origin xyz="0.411 0 0.311"/>
             <geometry>
-                <box size ="0.3 0.3 0.15"/>
+                <box size ="0.822 0.8 0.622"/>
             </geometry>
             <material name="white"/>
         </visual>
         <collision>
-            <origin xyz="0.15 0 0.075"/>
+            <origin xyz="0.411 0 0.311"/>
             <geometry>
-                <box size ="0.3 0.3 0.15"/>
+                <box size ="0.822 0.8 0.622"/>
             </geometry>
         </collision>
-        <xacro:inertial_box mass="0.5" x="0.3" y="0.3" z="0.15">
-            <origin xyz="-0.15 0 0.075" rpy="0 0 0"/>
+        <xacro:inertial_box mass="0.822" x="0.8" y="0.8" z="0.622">
+            <origin xyz="-0.411 0 0.311" rpy="0 0 0"/>
         </xacro:inertial_box>
     </link>

Commit message: change

File: description/robot_core.xacro (robot description, xacro)
@@ -53,5 +53,5 @@
         <parent link="base_link"/>
         <child link="left_wheel"/>
-        <origin xyz="0 0.175 0" rpy="-${pi/2} 0 0"/>
+        <origin xyz="0 0.822 0" rpy="-${pi/2} 0 0"/>
         <axis xyz="0 0 1"/>
     </joint>
@@ -75,5 +75,5 @@
         <parent link="base_link"/>
         <child link="right_wheel"/>
-        <origin xyz="0 -0.175 0" rpy="${pi/2} 0 0"/>
+        <origin xyz="0 -0.822 0" rpy="${pi/2} 0 0"/>
         <axis xyz="0 0 -1"/>
     </joint>

Commit message: change

File: description/robot_core.xacro (robot description, xacro)
@@ -53,5 +53,5 @@
         <parent link="base_link"/>
         <child link="left_wheel"/>
-        <origin xyz="0 0.822 0" rpy="-${pi/2} 0 0"/>
+        <origin xyz="0 0.412 0" rpy="-${pi/2} 0 0"/>
         <axis xyz="0 0 1"/>
     </joint>
@@ -75,5 +75,5 @@
         <parent link="base_link"/>
         <child link="right_wheel"/>
-        <origin xyz="0 -0.822 0" rpy="${pi/2} 0 0"/>
+        <origin xyz="0 -0.412 0" rpy="${pi/2} 0 0"/>
         <axis xyz="0 0 -1"/>
     </joint>

Commit message: change

File: description/robot_core.xacro (robot description, xacro)
@@ -75,5 +75,5 @@
         <parent link="base_link"/>
         <child link="right_wheel"/>
-        <origin xyz="0 -0.412 0" rpy="${pi/2} 0 0"/>
+        <origin xyz="0 -0.413 0" rpy="${pi/2} 0 0"/>
         <axis xyz="0 0 -1"/>
     </joint>
@@ -94,3 +94,49 @@
         </xacro:inertial_cylinder>
     </link>
+<!-- LEFT FRONT WHEEL LINK -->
+    <joint name="left_front_wheel_joint" type="continuous">
+        <parent link="base_link"/>
+        <child link="left_front_wheel"/>
+        <origin xyz="0.2 0.413 0" rpy="-${pi/2} 0 0"/>
+        <axis xyz="0 0 1"/>
+    </joint>
+    <link name="left_front_wheel">
+        <visual>
+            <geometry>
+                <cylinder radius ="0.05" length="0.04"/>
+        </geometry>
+        <material name="blue"/>
+    </visual>
+    <collision>
+        <geometry>
+            <cylinder radius ="0.05" length="0.04"/>
+        </geometry>
+    </collision>
+    <xacro:inertial_cylinder mass="0.1" length="0.04" radius="0.05">
+        <origin xyz="0 0 0" rpy="0 0 0"/>
+    </xacro:inertial_cylinder>
+</link>
+<!-- RIGHT FRONT WHEEL LINK -->
+    <joint name="right_front_wheel_joint" type="continuous">
+        <parent link="base_link"/>
+        <child link="right_front_wheel"/>
+        <origin xyz="0.2 -0.413 0" rpy="${pi/2} 0 0"/>
+        <axis xyz="0 0 -1"/>
+    </joint>
+    <link name="right_front_wheel">
+        <visual>
+            <geometry>
+                <cylinder radius ="0.05" length="0.04"/>
+            </geometry>
+            <material name="blue"/>
+    </visual>
+    <collision>
+        <geometry>
+            <cylinder radius ="0.05" length="0.04"/>
+        </geometry>
+    </collision>
+    <xacro:inertial_cylinder mass="0.1" length="0.04" radius="0.05">
+        <origin xyz="0 0 0" rpy="0 0 0"/>
+    </xacro:inertial_cylinder>
+</link>
 </robot>

Commit message: change

File: description/robot_core.xacro (robot description, xacro)
@@ -98,5 +98,5 @@
         <parent link="base_link"/>
         <child link="left_front_wheel"/>
-        <origin xyz="0.2 0.413 0" rpy="-${pi/2} 0 0"/>
+        <origin xyz="0.83 0.413 0" rpy="-${pi/2} 0 0"/>
         <axis xyz="0 0 1"/>
     </joint>
@@ -121,5 +121,5 @@
         <parent link="base_link"/>
         <child link="right_front_wheel"/>
-        <origin xyz="0.2 -0.413 0" rpy="${pi/2} 0 0"/>
+        <origin xyz="0.83 -0.413 0" rpy="${pi/2} 0 0"/>
         <axis xyz="0 0 -1"/>
     </joint>

Commit message: change

File: description/robot_core.xacro (robot description, xacro)
@@ -53,5 +53,5 @@
         <parent link="base_link"/>
         <child link="left_wheel"/>
-        <origin xyz="0 0.412 0" rpy="-${pi/2} 0 0"/>
+        <origin xyz="0 0.415 0" rpy="-${pi/2} 0 0"/>
         <axis xyz="0 0 1"/>
     </joint>
@@ -75,5 +75,5 @@
         <parent link="base_link"/>
         <child link="right_wheel"/>
-        <origin xyz="0 -0.413 0" rpy="${pi/2} 0 0"/>
+        <origin xyz="0 -0.415 0" rpy="${pi/2} 0 0"/>
         <axis xyz="0 0 -1"/>
     </joint>
@@ -98,5 +98,5 @@
         <parent link="base_link"/>
         <child link="left_front_wheel"/>
-        <origin xyz="0.83 0.413 0" rpy="-${pi/2} 0 0"/>
+        <origin xyz="0.80 0.415 0" rpy="-${pi/2} 0 0"/>
         <axis xyz="0 0 1"/>
     </joint>
@@ -121,5 +121,5 @@
         <parent link="base_link"/>
         <child link="right_front_wheel"/>
-        <origin xyz="0.83 -0.413 0" rpy="${pi/2} 0 0"/>
+        <origin xyz="0.80 -0.415 0" rpy="${pi/2} 0 0"/>
         <axis xyz="0 0 -1"/>
     </joint>

Commit message: change

File: description/robot_core.xacro (robot description, xacro)
@@ -49,4 +49,7 @@
         </xacro:inertial_box>
     </link>
+    <gazebo reference="chassis">
+        <material>Gazebo/White</material>
+    </gazebo>
     <!-- LEFT WHEEL LINK -->
     <joint name="left_wheel_joint" type="continuous">
@@ -72,4 +75,7 @@
         </xacro:inertial_cylinder>
     </link>
+    <gazebo reference="left_wheel">
+        <material>Gazebo/Blue</material>
+    </gazebo>
     <joint name="right_wheel_joint" type="continuous">
         <parent link="base_link"/>
@@ -94,4 +100,7 @@
         </xacro:inertial_cylinder>
     </link>
+    <gazebo reference="right_wheel">
+        <material>Gazebo/Blue</material>
+    </gazebo>
 <!-- LEFT FRONT WHEEL LINK -->
     <joint name="left_front_wheel_joint" type="continuous">
@@ -117,4 +126,7 @@
     </xacro:inertial_cylinder>
 </link>
+    <gazebo reference="left_front_wheel">
+        <material>Gazebo/Blue</material>
+    </gazebo>
 <!-- RIGHT FRONT WHEEL LINK -->
     <joint name="right_front_wheel_joint" type="continuous">
@@ -140,3 +152,6 @@
     </xacro:inertial_cylinder>
 </link>
+    <gazebo reference="right_front_wheel">
+        <material>Gazebo/Blue</material>
+    </gazebo>
 </robot>

Commit message: change

File: description/robot_core.xacro (robot description, xacro)
@@ -107,5 +107,5 @@
         <parent link="base_link"/>
         <child link="left_front_wheel"/>
-        <origin xyz="0.80 0.415 0" rpy="-${pi/2} 0 0"/>
+        <origin xyz="0.7 0.415 0" rpy="-${pi/2} 0 0"/>
         <axis xyz="0 0 1"/>
     </joint>
@@ -133,5 +133,5 @@
         <parent link="base_link"/>
         <child link="right_front_wheel"/>
-        <origin xyz="0.80 -0.415 0" rpy="${pi/2} 0 0"/>
+        <origin xyz="0.7 -0.415 0" rpy="${pi/2} 0 0"/>
         <axis xyz="0 0 -1"/>
     </joint>

Commit message: change

File: description/robot_core.xacro (robot description, xacro)
@@ -56,5 +56,5 @@
         <parent link="base_link"/>
         <child link="left_wheel"/>
-        <origin xyz="0 0.415 0" rpy="-${pi/2} 0 0"/>
+        <origin xyz="0 0.42 0" rpy="-${pi/2} 0 0"/>
         <axis xyz="0 0 1"/>
     </joint>
@@ -81,5 +81,5 @@
         <parent link="base_link"/>
         <child link="right_wheel"/>
-        <origin xyz="0 -0.415 0" rpy="${pi/2} 0 0"/>
+        <origin xyz="0 -0.42 0" rpy="${pi/2} 0 0"/>
         <axis xyz="0 0 -1"/>
     </joint>
@@ -107,5 +107,5 @@
         <parent link="base_link"/>
         <child link="left_front_wheel"/>
-        <origin xyz="0.7 0.415 0" rpy="-${pi/2} 0 0"/>
+        <origin xyz="0.7 0.42 0" rpy="-${pi/2} 0 0"/>
         <axis xyz="0 0 1"/>
     </joint>
@@ -133,5 +133,5 @@
         <parent link="base_link"/>
         <child link="right_front_wheel"/>
-        <origin xyz="0.7 -0.415 0" rpy="${pi/2} 0 0"/>
+        <origin xyz="0.7 -0.42 0" rpy="${pi/2} 0 0"/>
         <axis xyz="0 0 -1"/>
     </joint>

Commit message: change

File: description/robot_core.xacro (robot description, xacro)
@@ -107,5 +107,5 @@
         <parent link="base_link"/>
         <child link="left_front_wheel"/>
-        <origin xyz="0.7 0.42 0" rpy="-${pi/2} 0 0"/>
+        <origin xyz="0.6 0.42 0" rpy="-${pi/2} 0 0"/>
         <axis xyz="0 0 1"/>
     </joint>
@@ -133,5 +133,5 @@
         <parent link="base_link"/>
         <child link="right_front_wheel"/>
-        <origin xyz="0.7 -0.42 0" rpy="${pi/2} 0 0"/>
+        <origin xyz="0.6 -0.42 0" rpy="${pi/2} 0 0"/>
         <axis xyz="0 0 -1"/>
     </joint>

Commit message: change

File: description/robot_core.xacro (robot description, xacro)
@@ -39,5 +39,5 @@
         </collision>
         <xacro:inertial_box mass="0.5" x="0.822" y="0.8" z="0.3">
-            <origin xyz="-0.411 0 0.15" rpy="0 0 0"/>
+            <origin xyz="0.411 0 0.15" rpy="0 0 0"/>
         </xacro:inertial_box>
     </link>
