Commit message: change

File: description/robot_core.xacro (robot description, xacro)
@@ -96,54 +96,21 @@
         <material>Gazebo/Blue</material>
     </gazebo>
-<!-- LEFT FRONT WHEEL LINK -->
-    <joint name="left_front_wheel_joint" type="continuous">
-        <parent link="base_link"/>
-        <child link="left_front_wheel"/>
-        <origin xyz="0.6 0.43 0" rpy="-${pi/2} 0 0"/>
-        <axis xyz="0 0 1"/>
+    <joint name="caster_wheel_joint" type="fixed">
+        <parent link="chassis"/>
+        <child link="caster_wheel"/>
+        <origin xyz="0.24 0 0" rpy="0 0 0"/>
     </joint>
-    <link name="left_front_wheel">
+    <link name="caster_wheel">
         <visual>
             <geometry>
-                <cylinder radius ="0.07" length="0.04"/>
-        </geometry>
-        <material name="blue"/>
-    </visual>
-    <collision>
-        <geometry>
-            <cylinder radius ="0.07" length="0.04"/>
-        </geometry>
-    </collision>
-    <xacro:inertial_cylinder mass="0.1" length="0.04" radius="0.07">
-        <origin xyz="0 0 0" rpy="0 0 0"/>
-    </xacro:inertial_cylinder>
-</link>
-    <gazebo reference="left_front_wheel">
-        <material>Gazebo/Blue</material>
-    </gazebo>
-<!-- RIGHT FRONT WHEEL LINK -->
-    <joint name="right_front_wheel_joint" type="continuous">
-        <parent link="base_link"/>
-        <child link="right_front_wheel"/>
-        <origin xyz="0.6 -0.43 0" rpy="${pi/2} 0 0"/>
-        <axis xyz="0 0 -1"/>
-    </joint>
-    <link name="right_front_wheel">
-        <visual>
-            <geometry>
-                <cylinder radius ="0.07" length="0.04"/>
+                <sphere radius="0.05" />
             </geometry>
-            <material name="blue"/>
-    </visual>
-    <collision>
-        <geometry>
-            <cylinder radius ="0.07" length="0.04"/>
-        </geometry>
-    </collision>
-    <xacro:inertial_cylinder mass="0.1" length="0.04" radius="0.07">
-        <origin xyz="0 0 0" rpy="0 0 0"/>
-    </xacro:inertial_cylinder>
-</link>
-    <gazebo reference="right_front_wheel">
+            <material name="black"/>
+        </visual>
+        <xacro:inertial_sphere mass="0.1" radius="0.05">
+            <origin xyz="0 0 0" rpy="0 0 0"/>
+        </xacro:inertial_sphere>
+    </link>
+    <gazebo reference="caster_wheel">
         <material>Gazebo/Blue</material>
     </gazebo>

Commit message: change

File: description/robot_core.xacro (robot description, xacro)
@@ -113,5 +113,7 @@
     </link>
     <gazebo reference="caster_wheel">
-        <material>Gazebo/Blue</material>
+        <material>Gazebo/Black</material>
+        <mu1 value="0.001"/>
+        <mu2 value="0.001"/>
     </gazebo>
 </robot>

Commit message: change

File: description/robot_core.xacro (robot description, xacro)
@@ -99,5 +99,5 @@
         <parent link="chassis"/>
         <child link="caster_wheel"/>
-        <origin xyz="0.24 0 0" rpy="0 0 0"/>
+        <origin xyz="0.74 0 0" rpy="0 0 0"/>
     </joint>
     <link name="caster_wheel">

Commit message: change

File: description/robot_core.xacro (robot description, xacro)
@@ -104,5 +104,5 @@
         <visual>
             <geometry>
-                <sphere radius="0.05" />
+                <sphere radius="0.07" />
             </geometry>
             <material name="black"/>

Commit message: change

File: description/robot_core.xacro (robot description, xacro)
@@ -108,4 +108,10 @@
             <material name="black"/>
         </visual>
+        <collision>
+            <geometry>
+                <sphere radius="0.07" />
+            </geometry>
+            <material name="black"/>
+        </collision>
         <xacro:inertial_sphere mass="0.1" radius="0.07">
             <origin xyz="0 0 0" rpy="0 0 0"/>

Commit message: change

File: description/robot_core.xacro (robot description, xacro)
@@ -61,5 +61,5 @@
         <collision>
             <geometry>
-                <cylinder radius ="0.07" length="0.04"/>
+                <sphere radius ="0.07"/>
             </geometry>
         </collision>
@@ -86,5 +86,5 @@
         <collision>
             <geometry>
-                <cylinder radius ="0.07" length="0.04"/>
+                <sphere radius ="0.07"/>
             </geometry>
         </collision>
