Commit message: change

File: description/camera.xacro (robot description, xacro)
@@ -1,28 +1,26 @@
 <?xml version="1.0"?>
 <robot xmlns:xacro="http://www.ros.org/wiki/xacro" >
-    <joint name="laser_joint" type="fixed">
+    <joint name="camera_joint" type="fixed">
         <parent link="chassis"/>
-        <child link="laser_frame"/>
-        <origin xyz="0.1 0 0.32" rpy="0 0 0"/>
+        <child link="camera_link"/>
+        <origin xyz="0.827 0 0.01" rpy="0 0 0"/>
     </joint>
-    <link name="laser_frame">
+    <link name="camera_link">
         <visual>
             <geometry>
-                <cylinder radius ="0.05" length="0.04"/>
+                <box size="0.010 0.03 0.03"/>
             </geometry>
             <material name="red"/>
         </visual>
-        <collision>
-            <geometry>
-                <cylinder radius ="0.05" length="0.04"/>
-            </geometry>
-        </collision>
-        <xacro:inertial_cylinder mass="0.1" length="0.04" radius="0.05">
-            <origin xyz="0 0 0" rpy="0 0 0"/>
-        </xacro:inertial_cylinder>
     </link>
-    <gazebo reference="laser_frame">
+    <joint name="camera_optical_joint" type="fixed">
+        <parent link="camera_link"/>
+        <child link="camera_link_optical"/>
+        <origin xyz="0 0 0" rpy="${-pi/2} 0 ${-pi/2}"/>
+    </joint>
+    <link name="camera_link_optical"></link>
+    <gazebo reference="camera_link">
         <material>Gazebo/Red</material>
-        <sensor name="laser" type="ray">
+        <!-- <sensor name="laser" type="ray">
             <pose>0 0 0 0 0 0</pose>
             <visualize>true</visualize>
@@ -51,4 +49,4 @@
             </plugin>
         </sensor>
-    </gazebo>
+    </gazebo> -->
 </robot>

Commit message: change

File: description/camera.xacro (robot description, xacro)
@@ -4,10 +4,10 @@
         <parent link="chassis"/>
         <child link="camera_link"/>
-        <origin xyz="0.827 0 0.01" rpy="0 0 0"/>
+        <origin xyz="0.822 0 0.2794" rpy="0 0 0"/>
     </joint>
     <link name="camera_link">
         <visual>
             <geometry>
-                <box size="0.010 0.03 0.03"/>
+                <box size="0.02516 0.08970 0.02491"/>
             </geometry>
             <material name="red"/>
