Commit message: change

File: description/lidar.xacro (robot description, xacro)
@@ -7,4 +7,15 @@
     </joint>
     <link name="laser_frame">
+        <visual>
+            <geometry>
+                <cylinder radius ="0.05" length="0.04"/>
+            </geometry>
+            <material name="red"/>
+        </visual>
+        <collision>
+            <geometry>
+                <cylinder radius ="0.05" length="0.04"/>
+            </geometry>
+        </collision>
     </link>
 </robot>

File: description/robot_core.xacro (robot description, xacro)
@@ -12,4 +12,7 @@
     <material name="black">
         <color rgba="0 0 0 1"/>
+    </material>
+    <material name="red">
+        <color rgba="1 0 0 1"/>
     </material>
     <link name="base_link">

Commit message: change

File: description/lidar.xacro (robot description, xacro)
@@ -17,5 +17,6 @@
                 <cylinder radius ="0.05" length="0.04"/>
             </geometry>
-        </collision>
+        <collision>
+            <origin xyz="0 0 0" ryp="0 0 0"/>
     </link>
 </robot>

Commit message: change

File: description/lidar.xacro (robot description, xacro)
@@ -17,5 +17,5 @@
                 <cylinder radius ="0.05" length="0.04"/>
             </geometry>
-        <collision>
+        </collision>
             <origin xyz="0 0 0" ryp="0 0 0"/>
     </link>

Commit message: change

File: description/lidar.xacro (robot description, xacro)
@@ -18,5 +18,7 @@
             </geometry>
         </collision>
-            <origin xyz="0 0 0" ryp="0 0 0"/>
+        <xacro:inertial_cylinder mass="0.1" length="0.4" radius "0.05">
+            <origin xyz="0 0 0" rpy="0 0 0"/>
+        </xacro:inertial_cylinder>
     </link>
 </robot>

Commit message: change

File: description/lidar.xacro (robot description, xacro)
@@ -4,5 +4,5 @@
         <parent link="chassis"/>
         <child link="laser_frame"/>
-        <origin xyz="0.1 0 0.175" rpy="0 0 0"/>
+        <origin xyz="0.1 0 0.32" rpy="0 0 0"/>
     </joint>
     <link name="laser_frame">

Commit message: change

File: description/lidar.xacro (robot description, xacro)
@@ -4,5 +4,5 @@
         <parent link="chassis"/>
         <child link="laser_frame"/>
-        <origin xyz="0.1 0 0.32" rpy="0 0 0"/>
+        <origin xyz="0.1 0 0.9" rpy="0 0 0"/>
     </joint>
     <link name="laser_frame">

Commit message: change

File: description/lidar.xacro (robot description, xacro)
@@ -23,4 +23,5 @@
     </link>
     <gazebo reference= "laser_frame">
+        <material>Gazebo/Red</material>
         <sensor name="laser" type="ray">
         <pose> 0 0 0 0 0 0 <pose>

Commit message: vh

File: description/lidar.xacro (robot description, xacro)
@@ -4,5 +4,5 @@
         <parent link="chassis"/>
         <child link="laser_frame"/>
-        <origin xyz="0.1 0 0.9" rpy="0 0 0"/>
+        <origin xyz="0.1 0 0.68" rpy="0 0 0"/>
     </joint>
     <link name="laser_frame">

Commit message: change

File: description/lidar.xacro (robot description, xacro)
@@ -4,5 +4,5 @@
         <parent link="chassis"/>
         <child link="laser_frame"/>
-        <origin xyz="0.1 0 0.68" rpy="0 0 0"/>
+        <origin xyz="0.1 0 0.6" rpy="0 0 0"/>
     </joint>
     <link name="laser_frame">

File: description/robot.urdf.xacro (robot description, xacro)
@@ -3,3 +3,4 @@
     <xacro:include filename="robot_core.xacro" />
     <xacro:include filename="lidar.xacro" />
+    <xacro:include filename="gazebo_control.xacro"/>
 </robot>

Commit message: change

File: description/lidar.xacro (robot description, xacro)
@@ -4,5 +4,5 @@
         <parent link="chassis"/>
         <child link="laser_frame"/>
-        <origin xyz="0.1 0 0.6" rpy="0 0 0"/>
+        <origin xyz="0.1 0 0.64" rpy="0 0 0"/>
     </joint>
     <link name="laser_frame">
@@ -18,5 +18,5 @@
             </geometry>
         </collision>
-        <xacro:inertial_cylinder mass="0.1" length="0.4" radius="0.05">
+        <xacro:inertial_cylinder mass="0.1" length="0.04" radius="0.05">
             <origin xyz="0 0 0" rpy="0 0 0"/>
         </xacro:inertial_cylinder>

Commit message: change

File: description/lidar.xacro (robot description, xacro)
@@ -4,5 +4,5 @@
         <parent link="chassis"/>
         <child link="laser_frame"/>
-        <origin xyz="0.1 0 0.64" rpy="0 0 0"/>
+        <origin xyz="0.1 0 0.32" rpy="0 0 0"/>
     </joint>
     <link name="laser_frame">

Commit message: change

File: description/lidar.xacro (robot description, xacro)
@@ -4,10 +4,10 @@
         <parent link="chassis"/>
         <child link="laser_frame"/>
-        <origin xyz="0.1 0 0.32" rpy="0 0 0"/>
+        <origin xyz="0.409575 0 0.3" rpy="0 0 0"/>
     </joint>
     <link name="laser_frame">
         <visual>
             <geometry>
-                <cylinder radius ="0.05" length="0.04"/>
+                <cylinder radius ="0.05395" length="0.04"/>
             </geometry>
             <material name="red"/>
@@ -15,8 +15,8 @@
         <collision>
             <geometry>
-                <cylinder radius ="0.05" length="0.04"/>
+                <cylinder radius ="0.05395" length="0.04"/>
             </geometry>
         </collision>
-        <xacro:inertial_cylinder mass="0.1" length="0.04" radius="0.05">
+        <xacro:inertial_cylinder mass="0.1" length="0.04" radius="0.05395">
             <origin xyz="0 0 0" rpy="0 0 0"/>
         </xacro:inertial_cylinder>

Commit message: change

File: description/lidar.xacro (robot description, xacro)
@@ -4,5 +4,5 @@
         <parent link="chassis"/>
         <child link="laser_frame"/>
-        <origin xyz="0.409575 0 0.3" rpy="0 0 0"/>
+        <origin xyz="0.409575 0 0.32" rpy="0 0 0"/>
     </joint>
     <link name="laser_frame">
